Commit message: Added wheels to URDF.

File: moose_description/urdf/moose.urdf.xacro (robot description, xacro)
@@ -2,11 +2,14 @@
 <robot name="moose" xmlns:xacro="http://www.ros.org/wiki/xacro">
   <xacro:property name="PI" value="3.1415926535897931"/>
-  <xacro:property name="wheel_radius" value="0.06" />
-  <xacro:property name="wheel_width" value="0.25" />
-  <xacro:property name="wheel_mass" value="15" />
-  <xacro:property name="wheel_to_track_ratio" value="0.5962" />
-  <xacro:property name="axle_x_offset" value="0.457367" />
-  <xacro:property name="axle_y_offset" value="0.0" />
-  <xacro:property name="axle_z_offset" value="-0.012977" />
+  <xacro:property name="wheel_radius" value="0.3175" />
+  <xacro:property name="wheel_width" value="0.303" />
+  <xacro:property name="wheel_mass" value="16.8" />
+  <xacro:property name="front_axle_x_offset" value="1.0036" />
+  <xacro:property name="front_mid_axle_x_offset" value="0.33639" />
+  <xacro:property name="rear_mid_axle_x_offset" value="-0.33638" />
+  <xacro:property name="rear_axle_x_offset" value="-1.01123" />
+  <xacro:property name="axle_y_offset" value="0.6249" />
+  <xacro:property name="high_axle_z_offset" value="0.04115" />
+  <xacro:property name="low_axle_z_offset" value="0.01892" />
   <xacro:property name="chassis_length" value="2.9532" />
   <xacro:property name="chassis_width" value="1.416" />
@@ -30,5 +33,5 @@
   <material name="white"><color rgba="0.9 0.9 0.9 1.0" /></material>
   <material name="red"><color rgba="0.9 0.0 0.0 1.0" /></material>
-  <!-- <xacro:macro name="wheel" params="prefix side *joint_pose">
+  <xacro:macro name="wheel" params="prefix side *joint_pose">
     <link name="${prefix}_${side}_wheel_link">
       <inertial>
@@ -38,5 +41,5 @@
       </inertial>
       <visual>
-        <origin xyz="0 0 0" rpy="0 0 ${PI/2}"/>
+        <origin xyz="0 ${wheel_width/2} 0" rpy="${PI/2} 0 0"/>
         <geometry>
           <mesh filename="package://moose_description/meshes/wheel.stl" />
@@ -45,5 +48,5 @@
       </visual>
       <collision>
-        <origin xyz="0 0 0" rpy="${PI/2} 0 0"/>
+        <origin xyz="0 0 0" rpy="0 0 0"/>
         <geometry>
           <cylinder radius="${wheel_radius}" length="${wheel_width}"/>
@@ -51,42 +54,45 @@
       </collision>
     </link>
-    <joint name="${prefix}_${side}_wheel_joint" type="continuous">
-      <parent link="${side}_diff_unit_link"/>
-      <child link="${side}_${prefix}_wheel_link"/>
+    <joint name="${prefix}_${side}_wheel" type="continuous">
+      <parent link="chassis_link"/>
+      <child link="${prefix}_${side}_wheel_link"/>
       <xacro:insert_block name="joint_pose" />
       <axis xyz="0 1 0"/>
     </joint>
-    <gazebo reference="${side}_${prefix}_wheel_link">
-      <selfCollide>false</selfCollide>
-      <mu1>0.9</mu1>
-      <mu2>0.5</mu2>
-      <kp value="10000000.0" />
-      <kd value="10.0" />
-      <fdir1 value="1 0 0" />
-      <material>Gazebo/Grey</material>
-    </gazebo>
-    <transmission name="${side}_${prefix}_wheel_trans">
+    <transmission name="${prefix}_${side}_wheel_trans">
       <type>transmission_interface/SimpleTransmission</type>
-      <joint name="${side}_${prefix}_wheel_joint">
+      <joint name="${prefix}_${side}_wheel_joint">
         <hardwareInterface>VelocityJointInterface</hardwareInterface>
       </joint>
-      <actuator name="${side}_${prefix}_actuator">
+      <!-- <actuator name="${side}_${prefix}_actuator">
         <hardwareInterface>VelocityJointInterface</hardwareInterface>
         <mechanicalReduction>1</mechanicalReduction>
-      </actuator>
+      </actuator> -->
     </transmission>
-  </xacro:macro> -->
-  <!-- <xacro:wheel prefix="front" side="left">
-    <origin xyz="${axle_x_offset*1} ${axle_y_offset*1} ${axle_z_offset}" rpy="0 0 0" />
+  </xacro:macro>
+  <xacro:wheel prefix="front" side="left">
+    <origin xyz="${front_axle_x_offset} ${axle_y_offset*1} ${high_axle_z_offset}" rpy="0 0 0" />
+  </xacro:wheel>
+  <xacro:wheel prefix="front_mid" side="left">
+    <origin xyz="${front_mid_axle_x_offset} ${axle_y_offset*1} ${low_axle_z_offset}" rpy="0 0 0" />
   </xacro:wheel>
   <xacro:wheel prefix="front" side="right">
-    <origin xyz="${axle_x_offset*1} ${axle_y_offset*-1} ${axle_z_offset}" rpy="0 0 0" />
+    <origin xyz="${front_axle_x_offset} ${axle_y_offset*-1} ${high_axle_z_offset}" rpy="0 0 0" />
+  </xacro:wheel>
+  <xacro:wheel prefix="front_mid" side="right">
+    <origin xyz="${front_mid_axle_x_offset} ${axle_y_offset*-1} ${low_axle_z_offset}" rpy="0 0 0" />
   </xacro:wheel>
   <xacro:wheel prefix="rear" side="left">
-    <origin xyz="${axle_x_offset*-1} ${axle_y_offset*1} ${axle_z_offset}" rpy="0 0 0" />
+    <origin xyz="${rear_axle_x_offset} ${axle_y_offset*1} ${high_axle_z_offset}" rpy="0 0 0" />
+  </xacro:wheel>
+  <xacro:wheel prefix="rear_mid" side="left">
+    <origin xyz="${rear_mid_axle_x_offset} ${axle_y_offset*1} ${low_axle_z_offset}" rpy="0 0 0" />
   </xacro:wheel>
   <xacro:wheel prefix="rear" side="right">
-    <origin xyz="${axle_x_offset*-1} ${axle_y_offset*-1} ${axle_z_offset}" rpy="0 0 0" />
-  </xacro:wheel> -->
+    <origin xyz="${rear_axle_x_offset} ${axle_y_offset*-1} ${high_axle_z_offset}" rpy="0 0 0" />
+  </xacro:wheel>
+  <xacro:wheel prefix="rear_mid" side="right">
+    <origin xyz="${rear_mid_axle_x_offset} ${axle_y_offset*-1} ${low_axle_z_offset}" rpy="0 0 0" />
+  </xacro:wheel>
   <link name="base_link"></link>
   <joint name="base_link_joint" type="fixed">
@@ -146,5 +152,5 @@
         <mesh filename="package://moose_description/meshes/top-deck.stl" />
       </geometry>
-      <material name="white"><color rgba="0.9 0.9 0.9 1.0" /></material>
+      <material name="yellow" />
     </visual>
   </link>

Commit message: Updated collisions,

File: moose_description/urdf/moose.urdf.xacro (robot description, xacro)
@@ -48,5 +48,5 @@
       </visual>
       <collision>
-        <origin xyz="0 0 0" rpy="0 0 0"/>
+        <origin xyz="0 0 0" rpy="${PI/2} 0 0"/>
         <geometry>
           <cylinder radius="${wheel_radius}" length="${wheel_width}"/>
@@ -60,13 +60,22 @@
       <axis xyz="0 1 0"/>
     </joint>
+    <gazebo reference="${prefix}_${side}_wheel_link">
+      <selfCollide>false</selfCollide>
+      <mu1>0.3</mu1>
+      <mu2>0.3</mu2>
+      <kp value="10000000.0" />
+      <kd value="1.0" />
+      <fdir1 value="1 0 0" />
+      <material>Gazebo/Grey</material>
+    </gazebo>
     <transmission name="${prefix}_${side}_wheel_trans">
       <type>transmission_interface/SimpleTransmission</type>
-      <joint name="${prefix}_${side}_wheel_joint">
-        <hardwareInterface>VelocityJointInterface</hardwareInterface>
+      <joint name="${prefix}_${side}_wheel">
+        <hardwareInterface>hardware_interface/VelocityJointInterface</hardwareInterface>
       </joint>
-      <!-- <actuator name="${side}_${prefix}_actuator">
-        <hardwareInterface>VelocityJointInterface</hardwareInterface>
+      <actuator name="${side}_${prefix}_actuator">
+        <hardwareInterface>hardware_interface/VelocityJointInterface</hardwareInterface>
         <mechanicalReduction>1</mechanicalReduction>
-      </actuator> -->
+      </actuator>
     </transmission>
   </xacro:macro>
@@ -115,6 +124,20 @@
       <material name="dark_grey" />
     </visual>
-  </link>
-  <link name="drive_motor_link"></link>
+    <collision>
+      <geometry>
+        <mesh filename="package://moose_description/meshes/chassis-collision.stl" />
+      </geometry>
+    </collision>
+  </link>
+  <link name="drive_motor_link">
+    <inertial>
+      <origin xyz="0 0 0" rpy="0 0 0" />
+      <mass value="0.01" />
+      <inertia
+        ixx="0.01" ixy="0.0" ixz="0.0"
+        iyy="0.01" iyz="0.0"
+        izz="0.01" />
+    </inertial>
+  </link>
   <joint name="drive_motor" type="continuous">
     <origin xyz="0 0 0" rpy="0 0 0" />
@@ -131,5 +154,14 @@
     </actuator>
   </transmission>
-  <link name="steer_motor_link"></link>
+  <link name="steer_motor_link">
+    <inertial>
+      <origin xyz="0 0 0" rpy="0 0 0" />
+      <mass value="0.01" />
+      <inertia
+        ixx="0.01" ixy="0.0" ixz="0.0"
+        iyy="0.01" iyz="0.0"
+        izz="0.01" />
+    </inertial>
+  </link>
   <joint name="steer_motor" type="continuous">
     <origin xyz="0 0 0" rpy="0 0 0" />
@@ -148,5 +180,4 @@
   <link name="top_chassis_link">
     <visual>
-      <origin xyz="0 0 -0.52705" rpy="0 0 0"/>
       <geometry>
         <mesh filename="package://moose_description/meshes/top-deck.stl" />
@@ -154,5 +185,14 @@
       <material name="yellow" />
     </visual>
-  </link>
+    <collision>
+      <geometry>
+        <mesh filename="package://moose_description/meshes/top-deck-collision.stl" />
+      </geometry>
+    </collision>
+  </link>
+  <gazebo reference="top_chassis_link">
+      <selfCollide>false</selfCollide>
+      <material>Gazebo/Yellow</material>
+  </gazebo>
   <joint name="top_link_joint" type="fixed">
     <origin xyz="0 0 0.52705" rpy="0 0 0" />
@@ -171,4 +211,26 @@
     <parent link="top_chassis_link"/>
     <child link="rear_top_chassis_link" />
+  </joint>
+  <link name="generator_link">
+    <visual>
+      <geometry>
+        <mesh filename="package://moose_description/meshes/generator.stl" />
+      </geometry>
+      <material name="yellow" />
+    </visual>
+    <collision>
+      <geometry>
+        <mesh filename="package://moose_description/meshes/generator-collision.stl" />
+      </geometry>
+    </collision>
+  </link>
+  <gazebo reference="generator_link">
+      <selfCollide>false</selfCollide>
+      <material>Gazebo/Yellow</material>
+  </gazebo>
+  <joint name="generator_joint" type="fixed">
+    <origin xyz="-0.641204 0 0" rpy="0 0 0" />
+    <parent link="top_chassis_link"/>
+    <child link="generator_link" />
   </joint>
   <link name="imu_link" />

Commit message: Made the generator optional

File: moose_description/urdf/moose.urdf.xacro (robot description, xacro)
@@ -212,26 +212,28 @@
     <child link="rear_top_chassis_link" />
   </joint>
-  <link name="generator_link">
-    <visual>
-      <geometry>
-        <mesh filename="package://moose_description/meshes/generator.stl" />
-      </geometry>
-      <material name="yellow" />
-    </visual>
-    <collision>
-      <geometry>
-        <mesh filename="package://moose_description/meshes/generator-collision.stl" />
-      </geometry>
-    </collision>
-  </link>
-  <gazebo reference="generator_link">
-      <selfCollide>false</selfCollide>
-      <material>Gazebo/Yellow</material>
-  </gazebo>
-  <joint name="generator_joint" type="fixed">
-    <origin xyz="-0.641204 0 0" rpy="0 0 0" />
-    <parent link="top_chassis_link"/>
-    <child link="generator_link" />
-  </joint>
+  <xacro:if value="$(optenv MOOSE_GENERATOR 0)">
+    <link name="generator_link">
+      <visual>
+        <geometry>
+          <mesh filename="package://moose_description/meshes/generator.stl" />
+        </geometry>
+        <material name="yellow" />
+      </visual>
+      <collision>
+        <geometry>
+          <mesh filename="package://moose_description/meshes/generator-collision.stl" />
+        </geometry>
+      </collision>
+    </link>
+    <gazebo reference="generator_link">
+        <selfCollide>false</selfCollide>
+        <material>Gazebo/Yellow</material>
+    </gazebo>
+    <joint name="generator_joint" type="fixed">
+      <origin xyz="-0.641204 0 0" rpy="0 0 0" />
+      <parent link="top_chassis_link"/>
+      <child link="generator_link" />
+    </joint>
+  </xacro:if>
   <link name="imu_link" />
   <joint name="imu_link_joint" type="fixed">

Commit message: Description cleanup (#1)
* Updated collisions,

* Made the generator optional

* Moved interactive markers to manned control and removed joy

File: moose_description/urdf/moose.urdf.xacro (robot description, xacro)
@@ -48,5 +48,5 @@
       </visual>
       <collision>
-        <origin xyz="0 0 0" rpy="0 0 0"/>
+        <origin xyz="0 0 0" rpy="${PI/2} 0 0"/>
         <geometry>
           <cylinder radius="${wheel_radius}" length="${wheel_width}"/>
@@ -60,13 +60,22 @@
       <axis xyz="0 1 0"/>
     </joint>
+    <gazebo reference="${prefix}_${side}_wheel_link">
+      <selfCollide>false</selfCollide>
+      <mu1>0.3</mu1>
+      <mu2>0.3</mu2>
+      <kp value="10000000.0" />
+      <kd value="1.0" />
+      <fdir1 value="1 0 0" />
+      <material>Gazebo/Grey</material>
+    </gazebo>
     <transmission name="${prefix}_${side}_wheel_trans">
       <type>transmission_interface/SimpleTransmission</type>
-      <joint name="${prefix}_${side}_wheel_joint">
-        <hardwareInterface>VelocityJointInterface</hardwareInterface>
+      <joint name="${prefix}_${side}_wheel">
+        <hardwareInterface>hardware_interface/VelocityJointInterface</hardwareInterface>
       </joint>
-      <!-- <actuator name="${side}_${prefix}_actuator">
-        <hardwareInterface>VelocityJointInterface</hardwareInterface>
+      <actuator name="${side}_${prefix}_actuator">
+        <hardwareInterface>hardware_interface/VelocityJointInterface</hardwareInterface>
         <mechanicalReduction>1</mechanicalReduction>
-      </actuator> -->
+      </actuator>
     </transmission>
   </xacro:macro>
@@ -115,6 +124,20 @@
       <material name="dark_grey" />
     </visual>
-  </link>
-  <link name="drive_motor_link"></link>
+    <collision>
+      <geometry>
+        <mesh filename="package://moose_description/meshes/chassis-collision.stl" />
+      </geometry>
+    </collision>
+  </link>
+  <link name="drive_motor_link">
+    <inertial>
+      <origin xyz="0 0 0" rpy="0 0 0" />
+      <mass value="0.01" />
+      <inertia
+        ixx="0.01" ixy="0.0" ixz="0.0"
+        iyy="0.01" iyz="0.0"
+        izz="0.01" />
+    </inertial>
+  </link>
   <joint name="drive_motor" type="continuous">
     <origin xyz="0 0 0" rpy="0 0 0" />
@@ -131,5 +154,14 @@
     </actuator>
   </transmission>
-  <link name="steer_motor_link"></link>
+  <link name="steer_motor_link">
+    <inertial>
+      <origin xyz="0 0 0" rpy="0 0 0" />
+      <mass value="0.01" />
+      <inertia
+        ixx="0.01" ixy="0.0" ixz="0.0"
+        iyy="0.01" iyz="0.0"
+        izz="0.01" />
+    </inertial>
+  </link>
   <joint name="steer_motor" type="continuous">
     <origin xyz="0 0 0" rpy="0 0 0" />
@@ -148,5 +180,4 @@
   <link name="top_chassis_link">
     <visual>
-      <origin xyz="0 0 -0.52705" rpy="0 0 0"/>
       <geometry>
         <mesh filename="package://moose_description/meshes/top-deck.stl" />
@@ -154,5 +185,14 @@
       <material name="yellow" />
     </visual>
-  </link>
+    <collision>
+      <geometry>
+        <mesh filename="package://moose_description/meshes/top-deck-collision.stl" />
+      </geometry>
+    </collision>
+  </link>
+  <gazebo reference="top_chassis_link">
+      <selfCollide>false</selfCollide>
+      <material>Gazebo/Yellow</material>
+  </gazebo>
   <joint name="top_link_joint" type="fixed">
     <origin xyz="0 0 0.52705" rpy="0 0 0" />
@@ -172,4 +212,28 @@
     <child link="rear_top_chassis_link" />
   </joint>
+  <xacro:if value="$(optenv MOOSE_GENERATOR 0)">
+    <link name="generator_link">
+      <visual>
+        <geometry>
+          <mesh filename="package://moose_description/meshes/generator.stl" />
+        </geometry>
+        <material name="yellow" />
+      </visual>
+      <collision>
+        <geometry>
+          <mesh filename="package://moose_description/meshes/generator-collision.stl" />
+        </geometry>
+      </collision>
+    </link>
+    <gazebo reference="generator_link">
+        <selfCollide>false</selfCollide>
+        <material>Gazebo/Yellow</material>
+    </gazebo>
+    <joint name="generator_joint" type="fixed">
+      <origin xyz="-0.641204 0 0" rpy="0 0 0" />
+      <parent link="top_chassis_link"/>
+      <child link="generator_link" />
+    </joint>
+  </xacro:if>
   <link name="imu_link" />
   <joint name="imu_link_joint" type="fixed">
